File: KiCAD_project/zdc_fifo_test/zdc_fifo_test.kicad_sch (KiCad schematic)
At the start: 103 parts, among them IC1 OPA695IDR, J1 Conn_Coaxial, J2 Conn_Coaxial, J3 Conn_Coaxial, J4 Conn_Coaxial, J5 Conn_Coaxial, J6 Conn_Coaxial, J7 Conn_Coaxial, J8 Conn_Coaxial, U1 THS3491xDDA, U2 THS3491xDDA, U3 THS3491xDDA, U4 THS3491xDDA, U5 LM7805_TO220, U6 LM7905_TO220, U8 LM7915_TO220, U9 LM7815_TO220

Commit message: added KiCAD project and ad8009 config
Parts:
- removed C31, C32, C34, C35, C37, C38, C40, C41, C43, C44, C46, C47, C49, C50, C52, C53: 1n, symbol Device:C
- removed C33, C36, C39, C42, C45, C48, C51, C54: 1u, symbol Device:C
- removed J1, J2, J3, J4: Conn_Coaxial, symbol Connector:Conn_Coaxial
- removed R1, R12, R16, R8: 51, symbol Device:R
- removed R10, R11, R14, R15, R2, R3, R6, R7: 1.5k, symbol Device:R
- removed R13, R4, R5, R9: 26.8k, symbol Device:R
- removed U1, U2, U3, U4: THS3491xDDA, Package_SO:Texas_R-PDSO-G8_EP2.95x4.9mm_Mask2.4x3.1mm, symbol Amplifier_Operational:THS3491xDDA
- removed VR1: 3006P-1-502LF, 3006P_1, symbol Device:3006P-1-502LF
- added C55, C58, C63, C64, C69, C70, C75, C76: 1n, symbol Device:C
- added C56, C59, C62, C65, C68, C71, C74, C77: 100n, symbol Device:C
- added C57, C60, C61, C66, C67, C72, C73, C78: 1u, symbol Device:C
- added IC2, IC3, IC4, IC5: AD8009ARZ, Library_footprints:SOIC127P600X175-8N, symbol Amplifier_Current:AD8009ARZ
- added J10, J11, J12, J9: Conn_Coaxial, symbol Connector:Conn_Coaxial
- added R28, R35, R39, R43: 51, Resistor_SMD:R_0402_1005Metric, symbol Device:R
- added R29, R30, R33, R34, R37, R38, R41, R42: 250, Resistor_SMD:R_0402_1005Metric, symbol Device:R
- added R31, R32, R36, R40: 2k, Resistor_SMD:R_0402_1005Metric, symbol Device:R
- added VR2: 3006P-1-502LF, Library_footprints:3006P_1, symbol Device:3006P-1-502LF
- C1, C10, C11, C12, C13, C15, C16, C18, C19, C2, C4, C5, C6, C7, C9: footprint (none) -> Capacitor_SMD:C_0402_1005Metric
- C26, C29: value 1n -> 100n
- IC1: footprint SOIC127P600X175-8N -> Library_footprints:SOIC127P600X175-8N
- R17, R18, R19, R20, R21, R22, R23, R24, R25, R26, R27: footprint (none) -> Resistor_SMD:R_0402_1005Metric
Connections:
- net +5V: now also C55.1, C56.1, C57.1, C64.1, C65.1, C66.1, C70.1, C71.1, C72.1, C76.1, C77.1, C78.1, IC2.7 (+VS), IC3.7 (+VS), IC4.7 (+VS), IC5.7 (+VS), VR2.3 (CW)
- net -5V: now also C58.1, C59.1, C60.1, C61.1, C62.1, C63.1, C67.1, C68.1, C69.1, C73.1, C74.1, C75.1, IC2.4 (-VS), IC3.4 (-VS), IC4.4 (-VS), IC5.4 (-VS), VR2.1 (CCW)
- net GND: now also C55.2, C56.2, C57.2, C58.2, C59.2, C60.2, C61.2, C62.2, C63.2, C64.2, C65.2, C66.2, C67.2, C68.2, C69.2, C70.2, C71.2, C72.2, C73.2, C74.2, C75.2, C76.2, C77.2, C78.2, J10.2 (Ext), J11.2 (Ext), J12.2 (Ext), J9.2 (Ext), R30.1, R33.1, R37.1, R41.1
- net at IC1.6 (OUTPUT), R17.2, R18.1: now also IC2.3 (+IN), IC3.3 (+IN), IC4.3 (+IN), IC5.3 (+IN)
- new net: IC2.2 (-IN), R29.1, R30.2, R31.1
- new net: IC2.6 (OUT), R28.1, R29.2
- new net: IC3.2 (-IN), R32.1, R33.2, R34.1
- new net: R31.2, R32.2, R36.2, R40.2, VR2.2 (WIPER)
- new net: IC4.2 (-IN), R36.1, R37.2, R38.1
- new net: IC4.6 (OUT), R38.2, R39.1
- new net: IC5.6 (OUT), R42.2, R43.1
- new net: J12.1 (In), R43.2
- new net: IC5.2 (-IN), R40.1, R41.2, R42.1
- new net: IC3.6 (OUT), R34.2, R35.1
- new net: J10.1 (In), R35.2
- new net: J9.1 (In), R28.2
- new net: J11.1 (In), R39.2
Other:
- moved on the sheet: C1, C10, C11, C12, C13, C14, C15, C16, C17, C18, C19, C2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

Commit message: Started PCB layout
Parts:
- removed C14: 100u, symbol Device:C_Polarized
- removed C15, C18: 1n, Capacitor_SMD:C_0402_1005Metric, symbol Device:C
- removed C16, C19: 0.1n, Capacitor_SMD:C_0402_1005Metric, symbol Device:C
- removed C17: 10u, symbol Device:C_Polarized
- removed D1, D4, D5, D6: 1N4007, Diode_THT:D_DO-41_SOD81_P10.16mm_Horizontal, symbol Diode:1N4007
- removed J10, J11, J12, J5, J6, J7, J8, J9: Conn_Coaxial, symbol Connector:Conn_Coaxial
- removed U5: LM7805_TO220, Package_TO_SOT_THT:TO-220-3_Vertical, symbol Regulator_Linear:LM7805_TO220
- removed U6: LM7905_TO220, Package_TO_SOT_THT:TO-220-3_Vertical, symbol Regulator_Linear:LM7905_TO220
- removed U8: LM7915_TO220, Package_TO_SOT_THT:TO-220-3_Vertical, symbol Regulator_Linear:LM7915_TO220
- removed U9: LM7815_TO220, Package_TO_SOT_THT:TO-220-3_Vertical, symbol Regulator_Linear:LM7815_TO220
- added C31: 100u, Library_footprints:CAP-SMD_BD6.3-L6.6-W6.6-LS7.6-FD-1, symbol Device:C_Polarized
- added C32, C35: 1n, Capacitor_SMD:C_0402_1005Metric, symbol Device:C
- added C33, C36: 0.1n, Capacitor_SMD:C_0402_1005Metric, symbol Device:C
- added C34: 10u, Capacitor_SMD:C_0805_2012Metric, symbol Device:C_Polarized
- added IC6, IC7: L7905ACD2T-TR, Library_footprints:STB20N95K5, symbol Regulator_Linear:L7905ACD2T-TR
- added IC8, IC9: L7805ACD2T-TR, Library_footprints:L7805ACD2TTR, symbol Regulator_Linear:L7805ACD2T-TR
- added J1, J2, J3, J4, J5, J6, J7, J8: EPL.00.250.NTN, Library_footprints:CONN_EPK.00.250.NTN_LMO, symbol Connector:EPL.00.250.NTN
- added U1: ~, Library_footprints:CONN-TH_XY126V-5.0-3P, symbol Connector:XY126V-5.0-3P
- C11, C5: footprint Capacitor_SMD:C_0402_1005Metric -> Capacitor_SMD:C_0805_2012Metric
- C20: footprint (none) -> Library_footprints:CAP-SMD_BD6.3-L6.6-W6.6-LS7.6-FD-1; JLCPCB (none) -> C2836437
- C21, C22, C24, C25, C26, C28, C29, C55, C56, C58, C59, C62, C63, C64, C65, C68, C69, C70, C71, C74, C75, C76, C77: footprint (none) -> Capacitor_SMD:C_0402_1005Metric
- C23: footprint (none) -> Capacitor_SMD:C_0805_2012Metric; JLCPCB (none) -> C15850
- C27: footprint (none) -> Capacitor_SMD:C_0603_1608Metric; JLCPCB (none) -> C15849
- C3, C8: footprint (none) -> Library_footprints:CAP-SMD_BD6.3-L6.6-W6.6-LS7.6-FD-1
- C30, C57, C60, C61, C66, C67, C72, C73, C78: footprint (none) -> Capacitor_SMD:C_0603_1608Metric
Connections:
- net GND: now also C31.1, C32.1, C33.1, C34.1, C35.1, C36.1, IC6.1 (GND), IC7.1 (GND), IC8.2 (GND), IC9.2 (GND), J1.2, J1.3, J1.4, J1.5, J2.2, J2.3, J2.4, J2.5, J3.2, J3.3, J3.4, J3.5, J4.2, J4.3, J4.4, J4.5, J5.2, J5.3, J5.4, J5.5, J6.2, J6.3, J6.4, J6.5, J7.2, J7.3, J7.4, J7.5, J8.2, J8.3, J8.4, J8.5, U1.2
- net at R43.2: now also J5.1
- net at R24.1, R25.1: now also J3.1
- net at R22.1, R23.1: now also J1.1
- net at R35.2: now also J7.1
- net at R20.1, R21.1: now also J2.1
- net at R28.2: now also J8.1
- net at R39.2: now also J6.1
- net at R26.1, R27.1: now also J4.1
- net +15V renamed +5V_stg2
- net +5V_stg2: now also C55.1, C56.1, C57.1, C64.1, C65.1, C66.1, C70.1, C71.1, C72.1, C76.1, C77.1, C78.1, IC2.7 (+VS), IC3.7 (+VS), IC4.7 (+VS), IC5.7 (+VS), VR2.3 (CW), IC9.3 (OUTPUT)
- net +24V NIM renamed +12V_NIM
- net +12V_NIM: now also IC8.1 (INPUT), IC9.1 (INPUT), U1.1
- removed net +5V: C28.1, C29.1, C30.1, C55.1, C56.1, C57.1, C64.1, C65.1, C66.1, C70.1, C71.1, C72.1, C76.1, C77.1, C78.1, IC1.7 (+VS), IC1.8 (~{DIS}), IC2.7 (+VS), IC3.7 (+VS), IC4.7 (+VS), IC5.7 (+VS), VR2.3 (CW)
- net -15V renamed +5V_stg1
- net +5V_stg1: now also C28.1, C29.1, C30.1, IC1.7 (+VS), IC1.8 (~{DIS}), IC8.3 (OUTPUT); no longer C23.2, C24.2, C25.2
- net -24V NIM renamed -12V_NIM
- net -12V_NIM: now also C31.2, C32.2, C33.2, IC6.2 (IN), IC7.2 (IN), U1.3
- net -5V renamed -5V_stg2
- net -5V_stg2: now also C34.2, C35.2, C36.2, IC7.3 (OUT); no longer C2.1, C26.1, C27.1, IC1.4 (-VS)
- new net -5V_stg1: C2.1, C23.2, C24.2, C25.2, C26.1, C27.1, IC1.4 (-VS), IC6.3 (OUT)
Other:
- moved on the sheet: C1, C20, C21, C22, C23, C24, C25, C3, C4, C5, C6, C7

Commit message: first gerber generated
Parts:
- added C37, C38, C39, C40, C41: NM, Capacitor_SMD:C_0402_1005Metric_Pad0.74x0.62mm_HandSolder, symbol Device:C
- added R44, R45, R46, R47: 0, Resistor_SMD:R_0603_1608Metric_Pad0.98x0.95mm_HandSolder, symbol Device:R
- added VR1: 3224W-1-500E, Library_footprints:3224W1500E, symbol Device:3224W-1-500E
- C1, C10, C22, C33: value 0.1n -> 100n
- C12, C24, C35, C6: value 1n -> 100n
- C13, C25, C36, C7: value 0.1n -> 1n
- C20, C3, C31, C8: value 100u -> 10u; footprint Library_footprints:CAP-SMD_BD6.3-L6.6-W6.6-LS7.6-FD-1 -> Resistor_SMD:R_0805_2012Metric
- C21, C32, C9: value 1n -> 1u
- C4: value 1n -> 1u; footprint Capacitor_SMD:C_0402_1005Metric -> Resistor_SMD:R_0402_1005Metric
- R19: value 134 -> 100
- R20, R22, R24, R26, R28, R35, R39, R43: footprint Resistor_SMD:R_0402_1005Metric -> Resistor_SMD:R_0603_1608Metric
Connections:
- net GND: now also VR1.1 (CCW); no longer R19.1
- net at IC2.2 (-IN), R29.1, R30.2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: now also C40.2
- net at IC2.6 (OUT), R28.1, R29.2: now also C40.1
- net at IC3.2 (-IN), R32.1, R33.2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: now also C39.2
- net at IC4.2 (-IN), R36.1, R37.2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: now also C38.2
- net at IC4.6 (OUT), R38.2, R39.1: now also C38.1
- net at IC1.2 (INVERTING_INPUT), R18.2, R19.2: now also C41.2
- net at IC5.6 (OUT), R42.2, R43.1: now also C37.1
- net at IC5.2 (-IN), R40.1, R41.2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: now also C37.2
- net at IC3.6 (OUT), R34.2, R35.1: now also C39.1
- new net: IC2.3 (+IN), R47.2
- new net: C41.1, IC1.6 (OUTPUT), R17.2, R18.1, R44.1, R45.1, R46.1, R47.1
- new net: IC5.3 (+IN), R44.2
- new net: IC4.3 (+IN), R45.2
- new net: R19.1, VR1.2 (WIPER)
- new net: IC3.3 (+IN), R46.2
Other:
- note added: "10u 100n 1n"
- note added: "10u 1u 100n ingresso"
- note added: "check max power 0402 resistor"
- note added: "da abbassate a 70 circa (68 ohm) E il trimmer da 50 FATTO"
- moved on the sheet: R19

Commit message: Added updated BOM files and gerber
Parts:
- C20, C3, C31, C8: footprint Resistor_SMD:R_0805_2012Metric -> Capacitor_SMD:C_0805_2012Metric
- C21, C32, C9: footprint Capacitor_SMD:C_0402_1005Metric -> Capacitor_SMD:C_0603_1608Metric
- C37, C38, C39, C40, C41, J1, J2, J3, J4, J5, J6, J7, J8: now left out of the parts list
- C4: footprint Resistor_SMD:R_0402_1005Metric -> Capacitor_SMD:C_0603_1608Metric
- R17: value 123 -> 120
- R20, R22, R24, R26: value 50 -> 51
- R21, R23, R25, R27: value 50 -> 51; footprint Resistor_SMD:R_0402_1005Metric -> Resistor_SMD:R_0603_1608Metric
- R29, R30, R33, R34, R37, R38, R41, R42: value 250 -> 240
- R31, R32, R36, R40: value 2k -> 976
Other:
- note added: "Questo è da 1k"
- note added: "Questo è da 200ohm"
- note removed: "10u 100n 1n"
- note removed: "10u 1u 100n ingresso"
- note removed: "check max power 0402 resistor"
- note removed: "da abbassate a 70 circa (68 ohm) E il trimmer da 50 FATTO"
Changed lines of the file:
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@@
 		(comment 1 "Stefan Cristi Zugravel")
 	)
-	(text "da abbassate a 70 circa (68 ohm)\nE il trimmer da 50\nFATTO\n"
+	(text "Questo è da 200ohm\n"
 		(exclude_from_sim no)
-		(at 200.406 19.304 0)
+		(at 169.926 27.432 0)
 		(effects
 			(font
@@
 		)
 	)
-	(text "10u 100n 1n\n"
+	(text "Questo è da 1k"
 		(exclude_from_sim no)
-		(at 93.218 207.264 0)
-		(effects
-			(font
-				(size 1.27 1.27)
-			)
-		)
-	)
-	(text "check max power 0402 resistor\n"
-		(exclude_from_sim no)
-		(at 383.54 229.362 0)
-		(effects
-			(font
-				(size 1.27 1.27)
-			)
-		)
-	)
-	(text "10u 1u 100n ingresso"
-		(exclude_from_sim no)
-		(at 40.132 205.994 0)
+		(at 266.954 237.998 0)
 		(effects
 			(font
@@
 			)
 		)
-		(property "Value" "250"
+		(property "Value" "240"
 			(at 347.98 240.0299 0)
 			(effects
@@
 			)
 		)
-		(property "Value" "2k"
+		(property "Value" "976"
 			(at 287.02 171.45 90)
 			(effects
@@
 			)
 		)
-		(property "Value" "123"
+		(property "Value" "120"
 			(at 255.27 58.4199 0)
 			(effects
@@
 			)
 		)
-		(property "Value" "250"
+		(property "Value" "240"
 			(at 358.14 125.73 90)
 			(effects
@@
 			)
 		)
-		(property "Footprint" "Resistor_SMD:R_0805_2012Metric"
+		(property "Footprint" "Capacitor_SMD:C_0805_2012Metric"
 			(at 131.7752 217.17 0)
 			(effects
@@
 			)
 		)
-		(property "Value" "250"
+		(property "Value" "240"
 			(at 347.98 184.1499 0)
 			(effects
@@
 		(unit 1)
 		(exclude_from_sim no)
-		(in_bom yes)
+		(in_bom no)
 		(on_board yes)
 		(dnp no)
@@
 		(unit 1)
 		(exclude_from_sim no)
-		(in_bom yes)
+		(in_bom no)
 		(on_board yes)
 		(dnp no)
@@
 			)
 		)
-		(property "Value" "2k"
+		(property "Value" "976"
 			(at 287.02 227.33 90)
 			(effects
@@
 		(unit 1)
 		(exclude_from_sim no)
-		(in_bom yes)
+		(in_bom no)
 		(on_board yes)
 		(dnp no)
@@
 			)
 		)
-		(property "Footprint" "Resistor_SMD:R_0805_2012Metric"
+		(property "Footprint" "Capacitor_SMD:C_0805_2012Metric"
 			(at 23.8252 198.12 0)
 			(effects
@@
 			)
 		)
-		(property "Value" "250"
+		(property "Value" "240"
 			(at 347.98 69.8499 0)
 			(effects
@@
 			)
 		)
-		(property "Footprint" "Capacitor_SMD:C_0402_1005Metric"
+		(property "Footprint" "Capacitor_SMD:C_0603_1608Metric"
 			(at 35.2552 170.18 0)
 			(effects
@@
 			)
 		)
-		(property "Value" "250"
+		(property "Value" "240"
 			(at 358.14 181.61 90)
 			(effects
@@
 		(unit 1)
 		(exclude_from_sim no)
-		(in_bom yes)
+		(in_bom no)
 		(on_board yes)
 		(dnp no)
@@
 			)
 		)
-		(property "Value" "50"
+		(property "Value" "51"
 			(at 142.24 17.78 90)
 			(effects
@@
 			)
 		)
-		(property "Footprint" "Resistor_SMD:R_0402_1005Metric"
+		(property "Footprint" "Resistor_SMD:R_0603_1608Metric"
 			(at 142.24 23.368 90)
 			(effects
@@
 		(unit 1)
 		(exclude_from_sim no)
-		(in_bom yes)
+		(in_bom no)
 		(on_board yes)
 		(dnp no)
@@
 		(unit 1)
 		(exclude_from_sim no)
-		(in_bom yes)
+		(in_bom no)
 		(on_board yes)
 		(dnp no)
@@
 			)
 		)
-		(property "Value" "250"
+		(property "Value" "240"
 			(at 358.14 67.31 90)
 			(effects
@@
 			)
 		)
-		(property "Footprint" "Capacitor_SMD:C_0402_1005Metric"
+		(property "Footprint" "Capacitor_SMD:C_0603_1608Metric"
 			(at 35.2552 198.12 0)
 			(effects
@@
 			)
 		)
-		(property "Footprint" "Resistor_SMD:R_0805_2012Metric"
+		(property "Footprint" "Capacitor_SMD:C_0805_2012Metric"
 			(at 131.7752 162.56 0)
 			(effects
@@
 			)
 		)
-		(property "Value" "250"
+		(property "Value" "240"
 			(at 347.98 128.2699 0)
 			(effects
@@
 		(unit 1)
 		(exclude_from_sim no)
-		(in_bom yes)
+		(in_bom no)
 		(on_board yes)
 		(dnp no)
@@
 			)
 		)
-		(property "Footprint" "Capacitor_SMD:C_0402_1005Metric"
+		(property "Footprint" "Capacitor_SMD:C_0603_1608Metric"
 			(at 144.4752 162.56 0)
 			(effects
@@
 			)
 		)
-		(property "Value" "2k"
+		(property "Value" "976"
 			(at 287.02 57.15 90)
 			(effects
@@
 			)
 		)
-		(property "Value" "50"
+		(property "Value" "51"
 			(at 133.35 77.4699 0)
 			(effects
@@
 			)
 		)
-		(property "Value" "50"
+		(property "Value" "51"
 			(at 133.35 101.5999 0)
 			(effects
@@
 			)
 		)
-		(property "Value" "50"
+		(property "Value" "51"
 			(at 142.24 41.91 90)
 			(effects
@@
 			)
 		)
-		(property "Footprint" "Resistor_SMD:R_0402_1005Metric"
+		(property "Footprint" "Resistor_SMD:R_0603_1608Metric"
 			(at 142.24 47.498 90)
 			(effects
@@
 			)
 		)
-		(property "Footprint" "Resistor_SMD:R_0805_2012Metric"
+		(property "Footprint" "Capacitor_SMD:C_0805_2012Metric"
 			(at 23.8252 170.18 0)
 			(effects
@@
 		(unit 1)
 		(exclude_from_sim no)
-		(in_bom yes)
+		(in_bom no)
 		(on_board yes)
 		(dnp no)
@@
 			)
 		)
-		(property "Value" "50"
+		(property "Value" "51"
 			(at 133.35 29.2099 0)
 			(effects
@@
 			)
 		)
-		(property "Value" "50"
+		(property "Value" "51"
 			(at 142.24 90.17 90)
 			(effects
@@
 			)
 		)
-		(property "Footprint" "Resistor_SMD:R_0402_1005Metric"
+		(property "Footprint" "Resistor_SMD:R_0603_1608Metric"
 			(at 142.24 95.758 90)
 			(effects
@@
 		(unit 1)
 		(exclude_from_sim no)
-		(in_bom yes)
+		(in_bom no)
 		(on_board yes)
 		(dnp no)
@@
 			)
 		)
-		(property "Footprint" "Resistor_SMD:R_0402_1005Metric"
+		(property "Footprint" "Capacitor_SMD:C_0603_1608Metric"
 			(at 144.4752 217.17 0)
 			(effects
@@
 		(unit 1)
 		(exclude_from_sim no)
-		(in_bom yes)
+		(in_bom no)
 		(on_board yes)
 		(dnp no)
@@
 		(unit 1)
 		(exclude_from_sim no)
-		(in_bom yes)
+		(in_bom no)
 		(on_board yes)
 		(dnp no)
@@
 		(unit 1)
 		(exclude_from_sim no)
-		(in_bom yes)
+		(in_bom no)
 		(on_board yes)
 		(dnp no)
@@
 			)
 		)
-		(property "Value" "250"
+		(property "Value" "240"
 			(at 358.14 237.49 90)
 			(effects
@@
 			)
 		)
-		(property "Value" "2k"
+		(property "Value" "976"
 			(at 287.02 115.57 90)
 			(effects
@@
 			)
 		)
-		(property "Value" "50"
+		(property "Value" "51"
 			(at 142.24 66.04 90)
 			(effects
@@
 			)
 		)
-		(property "Footprint" "Resistor_SMD:R_0402_1005Metric"
+		(property "Footprint" "Resistor_SMD:R_0603_1608Metric"
 			(at 142.24 71.628 90)
 			(effects
@@
 		(unit 1)
 		(exclude_from_sim no)
-		(in_bom yes)
+		(in_bom no)
 		(on_board yes)
 		(dnp no)
@@
 			)
 		)
-		(property "Value" "50"
+		(property "Value" "51"
 			(at 133.35 53.3399 0)
 			(effects

Commit message: cleaned up files
Parts:
- added C42, C43, C44, C45, C46, C47: 10u, Capacitor_SMD:C_0805_2012Metric, symbol Device:C
Connections:
- net +12V_NIM: now also C45.1, C46.1, C47.1
- net -12V_NIM: now also C42.2, C43.2, C44.2
- net GND: now also C42.1, C43.1, C44.1, C45.2, C46.2, C47.2
Other:
- note added: "Questo è da 500 o 1k"
- note removed: "Questo è da 1k"
- moved on the sheet: U1

Commit message: added slides material
Parts:
- R18: value 402 -> 390; footprint Resistor_SMD:R_0402_1005Metric -> Resistor_SMD:R_0603_1608Metric
- R21, R23, R25, R27: value 51 -> 1k; footprint Resistor_SMD:R_0603_1608Metric -> Resistor_SMD:R_0402_1005Metric
- R29, R30, R33, R34, R37, R38, R41, R42: value 240 -> 220
- R31, R32, R36, R40: value 976 -> 1k
Changed lines of the file:
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@@
 			)
 		)
-		(property "Value" "240"
+		(property "Value" "220"
 			(at 347.98 240.0299 0)
 			(effects
@@
 			)
 		)
-		(property "Value" "976"
+		(property "Value" "1k"
 			(at 287.02 171.45 90)
 			(effects
@@
 			)
 		)
-		(property "Value" "240"
+		(property "Value" "220"
 			(at 358.14 125.73 90)
 			(effects
@@
 			)
 		)
-		(property "Value" "402"
+		(property "Value" "390"
 			(at 203.2 29.21 90)
 			(effects
@@
 			)
 		)
-		(property "Footprint" "Resistor_SMD:R_0402_1005Metric"
+		(property "Footprint" "Resistor_SMD:R_0603_1608Metric"
 			(at 203.2 31.242 90)
 			(effects
@@
 			)
 		)
-		(property "Value" "240"
+		(property "Value" "220"
 			(at 347.98 184.1499 0)
 			(effects
@@
 			)
 		)
-		(property "Value" "976"
+		(property "Value" "1k"
 			(at 287.02 227.33 90)
 			(effects
@@
 			)
 		)
-		(property "Value" "240"
+		(property "Value" "220"
 			(at 347.98 69.8499 0)
 			(effects
@@
 			)
 		)
-		(property "Value" "240"
+		(property "Value" "220"
 			(at 358.14 181.61 90)
 			(effects
@@
 			)
 		)
-		(property "Value" "51"
+		(property "Value" "1k"
 			(at 142.24 17.78 90)
 			(effects
@@
 			)
 		)
-		(property "Footprint" "Resistor_SMD:R_0603_1608Metric"
+		(property "Footprint" "Resistor_SMD:R_0402_1005Metric"
 			(at 142.24 23.368 90)
 			(effects
@@
 			)
 		)
-		(property "Value" "240"
+		(property "Value" "220"
 			(at 358.14 67.31 90)
 			(effects
@@
 			)
 		)
-		(property "Value" "240"
+		(property "Value" "220"
 			(at 347.98 128.2699 0)
 			(effects
@@
 			)
 		)
-		(property "Value" "976"
+		(property "Value" "1k"
 			(at 287.02 57.15 90)
 			(effects
@@
 			)
 		)
-		(property "Value" "51"
+		(property "Value" "1k"
 			(at 142.24 41.91 90)
 			(effects
@@
 			)
 		)
-		(property "Footprint" "Resistor_SMD:R_0603_1608Metric"
+		(property "Footprint" "Resistor_SMD:R_0402_1005Metric"
 			(at 142.24 47.498 90)
 			(effects
@@
 			)
 		)
-		(property "Value" "51"
+		(property "Value" "1k"
 			(at 142.24 90.17 90)
 			(effects
@@
 			)
 		)
-		(property "Footprint" "Resistor_SMD:R_0603_1608Metric"
+		(property "Footprint" "Resistor_SMD:R_0402_1005Metric"
 			(at 142.24 95.758 90)
 			(effects
@@
 			)
 		)
-		(property "Value" "240"
+		(property "Value" "220"
 			(at 358.14 237.49 90)
 			(effects
@@
 			)
 		)
-		(property "Value" "976"
+		(property "Value" "1k"
 			(at 287.02 115.57 90)
 			(effects
@@
 			)
 		)
-		(property "Value" "51"
+		(property "Value" "1k"
 			(at 142.24 66.04 90)
 			(effects
@@
 			)
 		)
-		(property "Footprint" "Resistor_SMD:R_0603_1608Metric"
+		(property "Footprint" "Resistor_SMD:R_0402_1005Metric"
 			(at 142.24 71.628 90)
 			(effects
