File: KiCAD_project/zdc_fifo_test/zdc_fifo_test.kicad_sch (KiCad schematic)
At the start: 126 parts, among them IC1 OPA695IDR, IC2 AD8009ARZ, IC3 AD8009ARZ, IC4 AD8009ARZ, IC5 AD8009ARZ, IC6 L7905ACD2T-TR, IC7 L7905ACD2T-TR, IC8 L7805ACD2T-TR, IC9 L7805ACD2T-TR, J1 EPL.00.250.NTN, J2 EPL.00.250.NTN, J3 EPL.00.250.NTN, J4 EPL.00.250.NTN, J5 EPL.00.250.NTN, J6 EPL.00.250.NTN, J7 EPL.00.250.NTN, J8 EPL.00.250.NTN

Commit message: sim oscillation
Parts:
- added C14, C15, C17: 15p, symbol Device:C
- added C16: 0p, symbol Device:C
- added C79: 10u, Capacitor_SMD:C_0603_1608Metric, symbol Device:C
- added C80: 5p, Capacitor_SMD:C_0603_1608Metric, symbol Device:C
- C37, C38, C39, C40: value NM -> 2.2p; now in the parts list
- C41: value NM -> 4.7p; now in the parts list
- R31: now not fitted; now left out of the parts list
- R44, R45, R46, R47: value 0 -> 0.01; now not fitted; now left out of the parts list
Connections:
- net GND: now also C14.2, C15.2, C16.2, C17.2, C79.2, C80.2
- net at C41.1, IC1.6 (OUTPUT), R17.2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: now also C80.1; no longer IC2.3 (+IN), IC3.3 (+IN), IC4.3 (+IN), IC5.3 (+IN), R44.2, R45.2, R46.2, R47.2
- net at R31.2, R32.2, R36.2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: now also C79.1
- net at J5.1, R1.1, R43.2: now also C17.1
- net at J7.1, R3.1, R35.2: now also C15.1
- net at J8.1, R28.2, R4.1: now also C14.1
- net at J6.1, R2.1, R39.2: now also C16.1
- new net: IC2.3 (+IN), R47.2
- new net: IC5.3 (+IN), R44.2
- new net: IC4.3 (+IN), R45.2
- new net: IC3.3 (+IN), R46.2
